File: Adafruit BME680.sch (EAGLE design)
At the start: 14 parts, among them Q1 2N7002D, U1 BME280, U2 MIC5225-3.3

Commit message: Updated PCB files
Parts:
- removed JP2: (no value), microbuilder:HEADER-1X770MIL
- removed Q1: 2N7002D, microbuilder:MOSFET-N_DUAL
- removed U$15, U$5: FIDUCIAL_1MM, microbuilder:FIDUCIAL_1MM
- removed U$7, U$8: MOUNTINGHOLE2.0, microbuilder:MOUNTINGHOLE2.0
- removed U1: BME280, microbuilder:BME280
- added C2: 10uF, microbuilder:CAP_CERAMIC0805-NOOUTLINE
- added CONN3, CONN4: STEMMA_I2C_QT, microbuilder:STEMMA_I2C_QT
- added D1: GREEN, microbuilder:LED0603_NOOUTLINE
- added FID3, FID4: FIDUCIAL_1MM, microbuilder:FIDUCIAL_1MM
- added IC1: BME680, adafruit_sensor:BME680
- added JP1: (no value), microbuilder:HEADER-1X770MIL
- added Q2: BSS138, microbuilder:MOSFET-N_DUAL
- added R5: 10K, microbuilder:RESISTOR_0603_NOOUT
- added SJ1: (no value), microbuilder:SOLDERJUMPER
- added U$1, U$17: MOUNTINGHOLE2.5, microbuilder:MOUNTINGHOLE2.5
- C1: value 10uF -> 0.1uF; device microbuilder:CAP_CERAMIC0805-NOOUTLINE -> microbuilder:CAP_CERAMIC0603_NO
- U2: value MIC5225-3.3 -> AP2112K-3.3
Connections:
- removed net VIN: C1.1, JP2.1, R3G$1.1, R3G$3.1, U2.EN, U2.IN
- new net N$1: D1.A, R1.2
- new net VCC: C2.1, CONN3G$1.V+, CONN4G$1.V+, JP1.1, R3G$1.1, R3G$3.1, U2.EN, U2.IN
- net 3.3V: now also C1.1, IC1.VDD, IC1.VDDIO, JP1.2, Q21.G, Q22.G, R1.1, R5.2; no longer JP2.2, Q1G$1.G, Q1G$2.G, R1.2, U1.VDD, U1.VDDIO
- net CS: now also JP1.7; no longer JP2.7
- net CS_3V: now also IC1.CSB, R5.1; no longer R1.1, U1.CSB
- net GND: now also C2.2, CONN3G$1.GND, CONN4G$1.GND, D1.C, IC1.GND, JP1.3, SJ1.2; no longer JP2.3, U1.GND
- net SCK/SCL: now also CONN3G$1.SCL, CONN4G$1.SCL, JP1.4, Q21.D; no longer JP2.4, Q1G$1.D
- net SCK_3V: now also IC1.SCK, Q21.S; no longer Q1G$1.S, U1.SCK
- net SDI/SDA: now also CONN3G$1.SDA, CONN4G$1.SDA, JP1.6, Q22.D; no longer JP2.6, Q1G$2.D
- net SDI_3V: now also IC1.SDI, Q22.S; no longer Q1G$2.S, U1.SDI
- net SDO/ADR: now also IC1.SDO, JP1.5, SJ1.1; no longer JP2.5, U1.SDO
Other:
- note added: "I2C Pullups"
- note added: "I2C Pullups & Shift"
- note added: "ON LED"
- note added: "Power supply"
- note added: "STEMMA/I2C Headers"
- note removed: "For I2C leave CSB pulled high (default value) SDI=SDA, SCK=SCL"
- note removed: "For SPI set CSB low at startup SDO=MISO, SDI=MOSI, SCK=SCK, CSB=CS/SSEL"
- note removed: "LEVEL SHIFTING (5V <--> 3V)"
- moved on the sheet: C1, C3, D2, R1, R3G$1, R3G$2, R3G$3, R3G$4, R4, U2
